Commit message: created class container for bridge map

File: uri_gazebo/urdf/iris.urdf.xacro (robot description, xacro)
@@ -7,10 +7,10 @@
 		<collision name='body'>
 			<geometry>
-				<mesh filename="package://uri_gazebo/meshes/iris_12_coll.dae" scale="1 1 1" />
+				<mesh filename="package://uri_gazebo/meshes/iris_collision.dae" scale="1 1 1" />
 			</geometry>
 		</collision>
 		<visual name='body'>
 			<geometry>
-				<mesh filename="package://uri_gazebo/meshes/iris_12.dae" scale="1 1 1" />
+				<mesh filename="package://uri_gazebo/meshes/iris.dae" scale="1 1 1" />
 			</geometry>
 		</visual>

Commit message: added world for shore follòwning and added laser scanner to iris in gz

File: uri_gazebo/urdf/iris.urdf.xacro (robot description, xacro)
@@ -29,5 +29,5 @@
 		<origin xyz="-0.01 0.15 0.06" rpy="0 ${-M_PI/10} ${M_PI/4}"/>
 	</xacro:generic_camera>
-	<xacro:include filename="generic_camera.urdf.xacro" />
+<!--	<xacro:include filename="generic_camera.urdf.xacro" />-->
 	<xacro:generic_camera name="right_camera" parent="base_link" ros_topic="camera_image" cam_info_topic="camera_info" update_rate="30" res_x="320" res_y="240" image_format="R8G8B8" hfov="${0.6/M_PI * 180.0}">
 		<origin xyz="-0.01 -0.15 0.06" rpy="0 ${-M_PI/10} ${-M_PI/4}"/>
@@ -35,11 +35,25 @@
 	<!-- Sonar Range Finder -->
 	<xacro:include filename="sonar_sensor.urdf.xacro" />
-	<xacro:sonar_sensor name="sonar" parent="base_link" ros_topic="sonar_distance" update_rate="30" min_range="0.01" max_range="25.0" field_of_view="0.01" ray_count="1">
+	<xacro:sonar_sensor name="sonar" parent="base_link" ros_topic="sonar_distance" update_rate="40" min_range="0.01" max_range="25.0" field_of_view="0.01" ray_count="1">
 		<origin xyz="-0.0 0.0 -0.07" rpy="0 ${M_PI/2} 0"/>
 	</xacro:sonar_sensor>
 	<!-- laser Range Finder -->
-<!--	<xacro:include filename="sonar_sensor.urdf.xacro" />
-	<xacro:sonar_sensor name="laser" parent="base_link" ros_topic="laser" update_rate="10" min_range="0.01" max_range="25.0" field_of_view="${4*M_PI/3}" ray_count="180">
-		<origin xyz="0.0 0.0 -0.05" rpy="0 ${M_PI/2} ${M_PI/4}"/>
-	</xacro:sonar_sensor>-->
+	<xacro:include filename="generic_laser.urdf.xacro" />
+	<xacro:generic_laser
+		name="hokuyo"
+		parent="base_link"
+		size_x="0.1" size_y="0.1" size_z="0.1"
+		ros_topic="hokuyo"
+		visualize_laser="true"
+		update_rate="30"
+		samples="720"
+		min_angle="-1.570796"
+		max_angle="1.570796"
+		range_min="0.1"
+		range_max="30.0"
+		range_res="0.01"
+		noise_mean="0.0"
+		noise_stddv="0.01">
+		<origin xyz="0.25 0.0 0.02" rpy="${M_PI/2} ${-M_PI/3} 0"/>
+	</xacro:generic_laser>
 </robot>

Commit message: 3D scan can be colected through hovering

File: uri_gazebo/urdf/iris.urdf.xacro (robot description, xacro)
@@ -31,10 +31,10 @@
 <!--	<xacro:include filename="generic_camera.urdf.xacro" />-->
 	<xacro:generic_camera name="right_camera" parent="base_link" ros_topic="camera_image" cam_info_topic="camera_info" update_rate="30" res_x="320" res_y="240" image_format="R8G8B8" hfov="${0.6/M_PI * 180.0}">
-		<origin xyz="-0.01 -0.15 0.06" rpy="0 ${-M_PI/10} ${-M_PI/4}"/>
+		<origin xyz="-0.01 -0.15 0.06" rpy="0.1 ${-M_PI/10} ${-M_PI/4}"/>
 	</xacro:generic_camera>
 	<!-- Sonar Range Finder -->
 	<xacro:include filename="sonar_sensor.urdf.xacro" />
 	<xacro:sonar_sensor name="sonar" parent="base_link" ros_topic="sonar_distance" update_rate="40" min_range="0.01" max_range="25.0" field_of_view="0.01" ray_count="1">
-		<origin xyz="-0.0 0.0 -0.07" rpy="0 ${M_PI/2} 0"/>
+		<origin xyz="-0.0 0.0 -0.07" rpy="0.1 ${M_PI/2} 0"/>
 	</xacro:sonar_sensor>
 	<!-- laser Range Finder -->
@@ -43,17 +43,17 @@
 		name="hokuyo"
 		parent="base_link"
-		size_x="0.1" size_y="0.1" size_z="0.1"
+		size_x="0.05" size_y="0.05" size_z="0.07"
 		ros_topic="hokuyo"
 		visualize_laser="true"
 		update_rate="30"
-		samples="720"
-		min_angle="-1.570796"
-		max_angle="1.570796"
+		samples="1080"
+		min_angle="-2.09439510239"
+		max_angle="2.09439510239"
 		range_min="0.1"
-		range_max="30.0"
+		range_max="10.0"
 		range_res="0.01"
 		noise_mean="0.0"
 		noise_stddv="0.01">
-		<origin xyz="0.25 0.0 0.02" rpy="${M_PI/2} ${-M_PI/3} 0"/>
+		<origin xyz="-0.02 0.0 0.18" rpy="${M_PI/2} ${-M_PI/2} 0"/>
 	</xacro:generic_laser>
 </robot>

Commit message: shore follwing working in simulation, bridge exploration working in simulation but need to be fixed in the update of the map/frotier

File: uri_gazebo/urdf/iris.urdf.xacro (robot description, xacro)
@@ -26,10 +26,10 @@
   <!-- MAPIP cameras -->
 	<xacro:include filename="generic_camera.urdf.xacro" />
-	<xacro:generic_camera name="left_camera" parent="base_link" ros_topic="camera_image" cam_info_topic="camera_info" update_rate="30" res_x="320" res_y="240" image_format="R8G8B8" hfov="${0.6/M_PI * 180.0}">
-		<origin xyz="-0.01 0.15 0.06" rpy="0 ${-M_PI/10} ${M_PI/4}"/>
+	<xacro:generic_camera name="left_camera" parent="base_link" ros_topic="camera_image" cam_info_topic="camera_info" update_rate="30" res_x="4608" res_y="3456" image_format="R8G8B8" hfov="${0.6/M_PI * 180.0}">
+		<origin xyz="-0.01 0.15 0.06" rpy="0 ${-M_PI/1000} ${M_PI/4}"/>
 	</xacro:generic_camera>
 <!--	<xacro:include filename="generic_camera.urdf.xacro" />-->
-	<xacro:generic_camera name="right_camera" parent="base_link" ros_topic="camera_image" cam_info_topic="camera_info" update_rate="30" res_x="320" res_y="240" image_format="R8G8B8" hfov="${0.6/M_PI * 180.0}">
-		<origin xyz="-0.01 -0.15 0.06" rpy="0.1 ${-M_PI/10} ${-M_PI/4}"/>
+	<xacro:generic_camera name="right_camera" parent="base_link" ros_topic="camera_image" cam_info_topic="camera_info" update_rate="30" res_x="4608" res_y="3456" image_format="R8G8B8" hfov="${0.6/M_PI * 180.0}">
+		<origin xyz="0.15 -0.15 0.06" rpy="0.0 0.01 0.0"/>
 	</xacro:generic_camera>
 	<!-- Sonar Range Finder -->

File: uri_gazebo/urdf/iris_2_cameras.urdf.xacro (robot description, xacro)
@@ -10,9 +10,9 @@
 	<!-- MAPIR cameras -->
 	<xacro:include filename="generic_camera.urdf.xacro" />
-	<xacro:generic_camera name="left_camera" parent="base_link" ros_topic="camera_image" cam_info_topic="camera_info" update_rate="30" res_x="320" res_y="240" image_format="R8G8B8" hfov="${0.6/M_PI * 180.0}">
-		<origin xyz="-0.01 0.15 0.06" rpy="0 ${-M_PI/10} ${M_PI/4}"/>
+	<xacro:generic_camera name="left_camera" parent="base_link" ros_topic="camera_image" cam_info_topic="camera_info" update_rate="30" res_x="4608" res_y="3456" image_format="R8G8B8" hfov="${0.6/M_PI * 180.0}">
+		<origin xyz="-0.01 0.15 0.06" rpy="0 ${-M_PI/1050} ${M_PI/4}"/>
 	</xacro:generic_camera>
-	<xacro:generic_camera name="right_camera" parent="base_link" ros_topic="camera_image" cam_info_topic="camera_info" update_rate="30" res_x="320" res_y="240" image_format="R8G8B8" hfov="${0.6/M_PI * 180.0}">
-		<origin xyz="-0.01 -0.15 0.06" rpy="0 ${-M_PI/10} ${-M_PI/4}"/>
+	<xacro:generic_camera name="right_camera" parent="base_link" ros_topic="camera_image" cam_info_topic="camera_info" update_rate="30" res_x="4608" res_y="3456" image_format="R8G8B8" hfov="${0.6/M_PI * 180.0}">
+		<origin xyz="-0.01 -0.15 0.06" rpy="0 ${-M_PI/1050} ${-M_PI/4}"/>
 	</xacro:generic_camera>
 	<!-- Sonar Range Finder -->

File: uri_shorefollowing/urdf/iris_laser_shore_following.urdf.xacro (robot description, xacro)
@@ -25,5 +25,5 @@
 		noise_mean="0.0"
 		noise_stddv="0.03">
-		<origin xyz="0.0 0.0 -0.10" rpy="0 ${M_PI/2} 0"/>
+		<origin xyz="0.0 0.0 -0.10" rpy="0 ${M_PI/3} 0"/>
 	</xacro:generic_laser>
 	<!-- Sonar Range Finder -->
